File: hardware/kicad/kicad.kicad_sch (KiCad schematic)
At the start: 4 parts, among them U1 RP2040

Commit message: [30-8] update progress
Parts:
- added C1, C2, C3, C4, C5: C, Capacitor_SMD:C_0603_1608Metric_Pad1.08x0.95mm_HandSolder, symbol Device:C
- added F1: Polyfuse, Fuse:Fuse_0603_1608Metric_Pad1.05x0.95mm_HandSolder, symbol Device:Polyfuse
- added J1: Conn_01x05, Connector_PinHeader_2.54mm:PinHeader_1x05_P2.54mm_Vertical, symbol Connector_Generic:Conn_01x05
- added J2: USB_C_Receptacle_USB2.0, Connector_USB:USB_C_Receptacle_HRO_TYPE-C-31-M-12, symbol Connector:USB_C_Receptacle_USB2.0
- added R4, R5, R6, R7: R, Resistor_SMD:R_0603_1608Metric_Pad0.98x0.95mm_HandSolder, symbol Device:R
- added SW1: SW_Push, Button_Switch_SMD:SW_SPST_TL3342, symbol Switch:SW_Push
- added U2: W25Q128JVS, Package_SO:SOIC-8_5.23x5.23mm_P1.27mm, symbol Memory_Flash:W25Q128JVS
- added U3: XC6206PxxxMR, Package_TO_SOT_SMD:SOT-23, symbol Regulator_Linear:XC6206PxxxMR
- added U4: USBLC6-2SC6, Package_TO_SOT_SMD:SOT-23-6, symbol Power_Protection:USBLC6-2SC6
- added Y1: Crystal_GND24_Small, Crystal:Crystal_SMD_3225-4Pin_3.2x2.5mm_HandSoldering, symbol Device:Crystal_GND24_Small
Connections:
- net +3V3: now also C1.2, C5.1, J1.2 (Pin_2), U2.8 (VCC), U3.2 (VO)
- net CS: now also R4.1, U2.1 (~{CS})
- net D_N: now also U4.3 (I/O2)
- net D_P: now also U4.1 (I/O1)
- net GND: now also C1.1, C2.2, C3.1, C4.1, C5.2, J1.3 (Pin_3), J2.A1 (GND), J2.A12 (GND), J2.B1 (GND), J2.B12 (GND), J2.S1 (SHIELD), R6.2, R7.2, SW1.1, U2.4 (GND), U3.1 (GND), U4.2 (GND), Y1.2, Y1.4
- net QSPI_CLK: now also U2.6 (CLK)
- net RESET: now also J1.1 (Pin_1)
- net SD0: now also U2.5 (DI(IO0))
- net SD1: now also U2.2 (DO(IO1))
- net SD2: now also U2.3 (IO2)
- net SD3: now also U2.7 (IO3)
- net SWCLK: now also J1.5 (Pin_5)
- net SWD: now also J1.4 (Pin_4)
- net XTAL_IN: now also C3.2, Y1.3
- net XTAL_OUT: now also R5.2
- new net: R4.2, SW1.2
- new net: C4.2, R5.1, Y1.1
- new net: J2.A5 (CC1), R6.1
- new net: J2.B5 (CC2), R7.1
- new net +5V: C2.1, F1.2, U3.3 (VI), U4.5 (VBUS)
- new net D_USB_N: J2.A7 (D-), J2.B7 (D-), U4.4 (I/O2)
- new net D_USB_P: J2.A6 (D+), J2.B6 (D+), U4.6 (I/O1)
- new net VBUS: F1.1, J2.A4 (VBUS), J2.A9 (VBUS), J2.B4 (VBUS), J2.B9 (VBUS)
- no-connect marks 0 -> 2
Other:
- moved on the sheet: R1, R2, R3, U1

Commit message: [1-9] update progress
Parts:
- added C10, C11, C12, C13, C14, C15, C6, C7, C8, C9: C, Capacitor_SMD:C_0603_1608Metric_Pad1.08x0.95mm_HandSolder, symbol Device:C
Connections:
- net +1V1: now also C6.1, C7.1, C8.1
- net +3V3: now also C10.1, C11.1, C12.1, C13.1, C14.1, C15.1, C9.1
- net CS: now also R4.2; no longer R4.1
- net GND: now also C10.2, C11.2, C12.2, C13.2, C14.2, C15.2, C6.2, C7.2, C8.2, C9.2
- net at SW1.2: now also R4.1; no longer R4.2
Other:
- moved on the sheet: C2, C3, C4, C5, J1, R4, R5, U3, Y1

Commit message: [16-09] added level shifter + progress on the expasion connector
Parts:
- added D1, D10, D11, D12, D13, D14, D15, D16, D17, D18, D19, D2, D20, D21, D22, D23, D24, D25, D26, D27, D28, D29, D3, D30, D31, D32, D33, D34, D35, D4, D5, D6, D7, D8, D9: 1N4148W, Diode_SMD:D_SOD-123, symbol Diode:1N4148W
- added J3: Conn_01x08, Connector_PinHeader_2.54mm:PinHeader_1x08_P2.54mm_Vertical_SMD_Pin1Right, symbol Connector_Generic:Conn_01x08
- added LED1, LED10, LED11, LED12, LED13, LED14, LED15, LED16, LED17, LED18, LED19, LED2, LED20, LED21, LED22, LED23, LED24, LED25, LED26, LED27, LED28, LED29, LED3, LED30, LED31, LED32, LED33, LED34, LED35, LED4, LED5, LED6, LED7, LED8, LED9: MX_SK6812MINI-E, marbastlib-mx:LED_MX_6028R, symbol marbastlib-mx:MX_SK6812MINI-E
- added QSel3: AO3400A, Package_TO_SOT_SMD:SOT-23, symbol Transistor_FET:AO3400A
- added QSel5: AO3401A, Package_TO_SOT_SMD:SOT-23, symbol Transistor_FET:AO3401A
- added RSel1: 5k1, Resistor_SMD:R_0603_1608Metric_Pad0.98x0.95mm_HandSolder, symbol Device:R
- added SW1, SW10, SW11, SW12, SW13, SW14, SW15, SW16, SW17, SW18, SW19, SW2, SW20, SW21, SW22, SW23, SW24, SW25, SW26, SW27, SW28, SW29, SW3, SW30, SW31, SW32, SW33, SW34, SW35, SW4, SW5, SW6, SW7, SW8, SW9: MX_SW_solder, marbastlib-mx:SW_MX_1u, symbol marbastlib-mx:MX_SW_solder
- added SWSel1: SW_DIP_x01, Button_Switch_SMD:SW_DIP_SPSTx01_Slide_6.7x4.1mm_W6.73mm_P2.54mm_LowProfile_JPin, symbol Switch:SW_DIP_x01
- added U5: 74HC595, soic:SOIC16, symbol 74xx:74HC595
- R4, R5: value R -> 1k
- R6, R7: value R -> 5k1
- renumbered SW1 to SWR1
Connections:
- net +3V3: now also LED1.1 (VDD), LED10.1 (VDD), LED11.1 (VDD), LED12.1 (VDD), LED13.1 (VDD), LED14.1 (VDD), LED15.1 (VDD), LED16.1 (VDD), LED17.1 (VDD), LED18.1 (VDD), LED19.1 (VDD), LED2.1 (VDD), LED20.1 (VDD), LED21.1 (VDD), LED22.1 (VDD), LED23.1 (VDD), LED24.1 (VDD), LED25.1 (VDD), LED26.1 (VDD), LED27.1 (VDD), LED28.1 (VDD), LED29.1 (VDD), LED3.1 (VDD), LED30.1 (VDD), LED31.1 (VDD), LED32.1 (VDD), LED33.1 (VDD), LED34.1 (VDD), LED35.1 (VDD), LED4.1 (VDD), LED5.1 (VDD), LED6.1 (VDD), LED7.1 (VDD), LED8.1 (VDD), LED9.1 (VDD), QSel3.2 (S), SWSel1.2, U5.16 (VCC)
- net +5V: now also QSel5.3 (D)
- net GND: now also J3.1 (Pin_1), LED1.4 (VSS), LED10.4 (VSS), LED11.4 (VSS), LED12.4 (VSS), LED13.4 (VSS), LED14.4 (VSS), LED15.4 (VSS), LED16.4 (VSS), LED17.4 (VSS), LED18.4 (VSS), LED19.4 (VSS), LED2.4 (VSS), LED20.4 (VSS), LED21.4 (VSS), LED22.4 (VSS), LED23.4 (VSS), LED24.4 (VSS), LED25.4 (VSS), LED26.4 (VSS), LED27.4 (VSS), LED28.4 (VSS), LED29.4 (VSS), LED3.4 (VSS), LED30.4 (VSS), LED31.4 (VSS), LED32.4 (VSS), LED33.4 (VSS), LED34.4 (VSS), LED35.4 (VSS), LED4.4 (VSS), LED5.4 (VSS), LED6.4 (VSS), LED7.4 (VSS), LED8.4 (VSS), LED9.4 (VSS), RSel1.1, U5.10 (~{SRCLR}), U5.13 (~{OE}), U5.8 (GND)
- net GP8: now reaches U1.11 (GPIO8)
- net GP9: now reaches U1.12 (GPIO9)
- net GP10: now reaches U1.13 (GPIO10)
- net GP11: now reaches U1.14 (GPIO11)
- net GP12: now reaches U1.15 (GPIO12)
- net GP13: now reaches U1.16 (GPIO13)
- net GP14: now reaches U1.17 (GPIO14)
- net GP15: now reaches U1.18 (GPIO15)
- net LATCH: now reaches U1.2 (GPIO0)
- net LATCH: now also U5.12 (RCLK)
- net GP16: now reaches U1.27 (GPIO16)
- net GP17: now reaches U1.28 (GPIO17)
- net GP18: now reaches U1.29 (GPIO18)
- net SHIFT: now reaches U1.3 (GPIO1)
- net SHIFT: now also U5.11 (SRCLK)
- net GP19: now reaches U1.30 (GPIO19)
- net GP20: now reaches U1.31 (GPIO20)
- net GP21: now reaches U1.32 (GPIO21)
- net GP22: now reaches U1.34 (GPIO22)
- net GP23: now reaches U1.35 (GPIO23)
- net GP24: now reaches U1.36 (GPIO24)
- net GP25: now reaches U1.37 (GPIO25)
- net ADC0: now reaches U1.38 (GPIO26_ADC0)
- net ADC0: now also J3.7 (Pin_7)
- net ADC1: now reaches U1.39 (GPIO27_ADC1)
- net ADC1: now also J3.6 (Pin_6)
- net COLS: now reaches U1.4 (GPIO2)
- net COLS: now also U5.9 (QH')
- net ADC2: now reaches U1.40 (GPIO28_ADC2)
- net ADC3: now reaches U1.41 (GPIO29_ADC3)
- net ROW0: now reaches U1.5 (GPIO3)
- net ROW0: now also SW1.2, SW11.2, SW16.2, SW21.2, SW26.2, SW31.2, SW6.2
- net ROW1: now reaches U1.6 (GPIO4)
- net ROW1: now also SW12.2, SW17.2, SW2.2, SW22.2, SW27.2, SW32.2, SW7.2
- net ROW2: now reaches U1.7 (GPIO5)
- net ROW2: now also SW13.2, SW18.2, SW23.2, SW28.2, SW3.2, SW33.2, SW8.2
- net ROW3: now reaches U1.8 (GPIO6)
- net ROW3: now also SW14.2, SW19.2, SW24.2, SW29.2, SW34.2, SW4.2, SW9.2
- net ROW4: now reaches U1.9 (GPIO7)
- net ROW4: now also SW10.2, SW15.2, SW20.2, SW25.2, SW30.2, SW35.2, SW5.2
- new net: LED11.3 (DIN), LED6.2 (DOUT)
- new net: LED1.2 (DOUT), LED6.3 (DIN)
- new net: D20.2 (A), SW20.1
- new net: D31.2 (A), SW31.1
- new net: D13.2 (A), SW13.1
- new net: QSel3.1 (G), QSel5.1 (G), RSel1.2, SWSel1.1
- new net: J3.8 (Pin_8), QSel3.3 (D), QSel5.2 (S)
- new net: D19.2 (A), SW19.1
- new net: LED2.2 (DOUT), LED7.3 (DIN)
- new net: LED2.3 (DIN), LED31.2 (DOUT)
- new net: LED17.2 (DOUT), LED22.3 (DIN)
- new net: LED12.2 (DOUT), LED17.3 (DIN)
- new net: D11.2 (A), SW11.1
- new net: D3.2 (A), SW3.1
- new net: D25.2 (A), SW25.1
- new net: LED18.2 (DOUT), LED23.3 (DIN)
- new net: LED13.2 (DOUT), LED18.3 (DIN)
- new net: D14.2 (A), SW14.1
- new net: D16.2 (A), SW16.1
- new net: LED30.2 (DOUT), LED35.3 (DIN)
- new net: LED23.2 (DOUT), LED28.3 (DIN)
- new net: D6.2 (A), SW6.1
- new net: LED29.2 (DOUT), LED34.3 (DIN)
- new net: LED24.2 (DOUT), LED29.3 (DIN)
- new net: D30.2 (A), SW30.1
- new net: D4.2 (A), SW4.1
- new net: LED21.2 (DOUT), LED26.3 (DIN)
- new net: LED16.2 (DOUT), LED21.3 (DIN)
- new net: D33.2 (A), SW33.1
- new net: LED33.2 (DOUT), LED4.3 (DIN)
- new net: LED28.2 (DOUT), LED33.3 (DIN)
- new net: D17.2 (A), SW17.1
- new net: LED26.2 (DOUT), LED31.3 (DIN)
- new net: D1.2 (A), SW1.1
- new net: D22.2 (A), SW22.1
- new net: LED25.2 (DOUT), LED30.3 (DIN)
- new net: LED20.2 (DOUT), LED25.3 (DIN)
- new net: LED22.2 (DOUT), LED27.3 (DIN)
- new net: D28.2 (A), SW28.1
- new net: D8.2 (A), SW8.1
- new net: D10.2 (A), SW10.1
- new net: LED10.2 (DOUT), LED15.3 (DIN)
- new net: LED10.3 (DIN), LED5.2 (DOUT)
- new net: D26.2 (A), SW26.1
- new net: D35.2 (A), SW35.1
- new net: LED14.2 (DOUT), LED19.3 (DIN)
- new net: LED14.3 (DIN), LED9.2 (DOUT)
- new net: D21.2 (A), SW21.1
- new net: D9.2 (A), SW9.1
- new net: D34.2 (A), SW34.1
- new net: D2.2 (A), SW2.1
- new net: D27.2 (A), SW27.1
- new net: LED15.2 (DOUT), LED20.3 (DIN)
- new net: LED12.3 (DIN), LED7.2 (DOUT)
- new net: LED3.3 (DIN), LED32.2 (DOUT)
- new net: LED27.2 (DOUT), LED32.3 (DIN)
- new net: D24.2 (A), SW24.1
- new net: D18.2 (A), SW18.1
- new net: D15.2 (A), SW15.1
- new net: LED13.3 (DIN), LED8.2 (DOUT)
- new net: LED3.2 (DOUT), LED8.3 (DIN)
- new net: D12.2 (A), SW12.1
- new net: D32.2 (A), SW32.1
- new net: D23.2 (A), SW23.1
- new net: LED19.2 (DOUT), LED24.3 (DIN)
- new net: LED4.2 (DOUT), LED9.3 (DIN)
- new net: D7.2 (A), SW7.1
- new net: LED34.2 (DOUT), LED5.3 (DIN)
- new net: LED11.2 (DOUT), LED16.3 (DIN)
- new net: D29.2 (A), SW29.1
- new net: D5.2 (A), SW5.1
- new net COL0: D1.1 (K), D2.1 (K), D3.1 (K), D4.1 (K), D5.1 (K), U5.1 (QB)
- new net COL1: D10.1 (K), D6.1 (K), D7.1 (K), D8.1 (K), D9.1 (K), U5.2 (QC)
- new net COL2: D11.1 (K), D12.1 (K), D13.1 (K), D14.1 (K), D15.1 (K), U5.3 (QD)
- new net COL3: D16.1 (K), D17.1 (K), D18.1 (K), D19.1 (K), D20.1 (K), U5.4 (QE)
- new net COL4: D21.1 (K), D22.1 (K), D23.1 (K), D24.1 (K), D25.1 (K), U5.5 (QF)
- new net COL5: D26.1 (K), D27.1 (K), D28.1 (K), D29.1 (K), D30.1 (K), U5.6 (QG)
- new net COL6: D31.1 (K), D32.1 (K), D33.1 (K), D34.1 (K), D35.1 (K), U5.7 (QH)
- new net WS2812: LED1.3 (DIN)
Other:
- moved on the sheet: C10, C11, C12, C13, C14, C15, C3, C4, C9, F1, J2, R5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

Commit message: Update PCB
Parts:
- removed C1, C10, C11, C12, C13, C14, C15, C2, C3, C4, C5, C6, C7, C8, C9: C, Capacitor_SMD:C_0603_1608Metric_Pad1.08x0.95mm_HandSolder, symbol Device:C
- removed D1, D10, D11, D12, D13, D14, D15, D16, D17, D18, D19, D2, D20, D21, D22, D23, D24, D25, D26, D27, D28, D29, D3, D30, D31, D32, D33, D34, D35, D4, D5, D6, D7, D8, D9: 1N4148W, Diode_SMD:D_SOD-123, symbol Diode:1N4148W
- removed F1: Polyfuse, Fuse:Fuse_0603_1608Metric_Pad1.05x0.95mm_HandSolder, symbol Device:Polyfuse
- removed J1: Conn_01x05, Connector_PinHeader_2.54mm:PinHeader_1x05_P2.54mm_Vertical, symbol Connector_Generic:Conn_01x05
- removed J2: USB_C_Receptacle_USB2.0, Connector_USB:USB_C_Receptacle_HRO_TYPE-C-31-M-12, symbol Connector:USB_C_Receptacle_USB2.0
- removed J3: Conn_01x08, Connector_PinHeader_2.54mm:PinHeader_1x08_P2.54mm_Vertical_SMD_Pin1Right, symbol Connector_Generic:Conn_01x08
- removed LED32, LED33, LED34, LED35: MX_SK6812MINI-E, marbastlib-mx:LED_MX_6028R, symbol marbastlib-mx:MX_SK6812MINI-E
- removed QSel3: AO3400A, Package_TO_SOT_SMD:SOT-23, symbol Transistor_FET:AO3400A
- removed QSel5: AO3401A, Package_TO_SOT_SMD:SOT-23, symbol Transistor_FET:AO3401A
- removed R1, R4, R5: 1k, Resistor_SMD:R_0603_1608Metric_Pad0.98x0.95mm_HandSolder, symbol Device:R
- removed R2, R3: 27R, Resistor_SMD:R_0603_1608Metric_Pad0.98x0.95mm_HandSolder, symbol Device:R
- removed R6, R7, RSel1: 5k1, Resistor_SMD:R_0603_1608Metric_Pad0.98x0.95mm_HandSolder, symbol Device:R
- removed SW1, SW10, SW11, SW12, SW13, SW14, SW15, SW16, SW17, SW18, SW19, SW2, SW20, SW21, SW22, SW23, SW24, SW25, SW26, SW27, SW28, SW29, SW3, SW30, SW31, SW32, SW33, SW34, SW35, SW4, SW5, SW6, SW7, SW8, SW9: MX_SW_solder, marbastlib-mx:SW_MX_1u, symbol marbastlib-mx:MX_SW_solder
- removed SWR1: SW_Push, Button_Switch_SMD:SW_SPST_TL3342, symbol Switch:SW_Push
- removed SWSel1: SW_DIP_x01, Button_Switch_SMD:SW_DIP_SPSTx01_Slide_6.7x4.1mm_W6.73mm_P2.54mm_LowProfile_JPin, symbol Switch:SW_DIP_x01
- removed U1: RP2040, Package_DFN_QFN:QFN-56-1EP_7x7mm_P0.4mm_EP3.2x3.2mm, symbol MCU_RaspberryPi:RP2040
- removed U2: W25Q128JVS, Package_SO:SOIC-8_5.23x5.23mm_P1.27mm, symbol Memory_Flash:W25Q128JVS
- removed U3: XC6206PxxxMR, Package_TO_SOT_SMD:SOT-23, symbol Regulator_Linear:XC6206PxxxMR
- removed U4: USBLC6-2SC6, Package_TO_SOT_SMD:SOT-23-6, symbol Power_Protection:USBLC6-2SC6
- removed U5: 74HC595, soic:SOIC16, symbol 74xx:74HC595
- removed Y1: Crystal_GND24_Small, Crystal:Crystal_SMD_3225-4Pin_3.2x2.5mm_HandSoldering, symbol Device:Crystal_GND24_Small
- added J1: Conn_01x13_Female, Connector_PinHeader_1.00mm:PinHeader_1x13_P1.00mm_Vertical, symbol Connector:Conn_01x13_Female
- added LED0: MX_SK6812MINI-E, marbastlib-mx:LED_MX_6028R, symbol marbastlib-mx:MX_SK6812MINI-E
- added R0, R1, R10, R11, R12, R13, R14, R15, R16, R17, R18, R19, R2, R20, R21, R22, R23, R24, R25, R26, R27, R28, R29, R3, R30, R31, R4, R5, R6, R7, R8, R9: R_Small, Resistor_SMD:R_1206_3216Metric_Pad1.30x1.75mm_HandSolder, symbol Device:R_Small
- added SW0, SW1, SW10, SW11, SW12, SW13, SW14, SW15, SW16, SW17, SW18, SW19, SW2, SW20, SW21, SW22, SW23, SW24, SW25, SW26, SW27, SW28, SW29, SW3, SW30, SW31, SW4, SW5, SW6, SW7, SW8, SW9: MX_SW, marbastlib-mx:SW_MX_1u, symbol marbastlib-mx:MX_SW_HS
- added U1: Pico, MCU_RaspberryPi_and_Boards:RPi_Pico_SMD_TH, symbol MCU_RaspberryPi_and_Boards:Pico
- added U2, U3, U4, U5: MC74HC589ADR2G, Package_SO:SO-16_3.9x9.9mm_P1.27mm, symbol my_components:MC74HC589ADR2G
- added U6: ILI9163, my_components:ILI9163, symbol my_components:ILI9163
- added U7: ILI9341_TS, my_components:ILI9341_TS, symbol my_components:ILI9341_TS
- added USIPO0, USIPO1, USIPO2: 74HC595, Package_SO:SO-16_3.9x9.9mm_P1.27mm, symbol 74xx:74HC595
Connections:
- net +3V3: now also J1.1 (Pin_1), LED0.1 (VDD), SW0.1, SW1.1, SW10.1, SW11.1, SW12.1, SW13.1, SW14.1, SW15.1, SW16.1, SW17.1, SW18.1, SW19.1, SW2.1, SW20.1, SW21.1, SW22.1, SW23.1, SW24.1, SW25.1, SW26.1, SW27.1, SW28.1, SW29.1, SW3.1, SW30.1, SW31.1, SW4.1, SW5.1, SW6.1, SW7.1, SW8.1, SW9.1, U1.36 (3V3), U2.16 (VCC), U3.16 (VCC), U4.16 (VCC), U5.16 (VCC), U6.1 (LED), U6.8 (VCC), U7.14 (VCC), U7.7 (LED), USIPO0.10 (~{SRCLR}), USIPO0.16 (VCC), USIPO1.10 (~{SRCLR}), USIPO1.16 (VCC), USIPO2.10 (~{SRCLR}), USIPO2.16 (VCC)
- net GND: now also J1.3 (Pin_3), LED0.4 (VSS), R0.1, R1.1, R10.1, R11.1, R12.1, R13.1, R14.1, R15.1, R16.1, R17.1, R18.1, R19.1, R2.1, R20.1, R21.1, R22.1, R23.1, R24.1, R25.1, R26.1, R27.1, R28.1, R29.1, R3.1, R30.1, R31.1, R4.1, R5.1, R6.1, R7.1, R8.1, R9.1, U1.13 (GND), U1.18 (GND), U1.23 (GND), U1.28 (GND), U1.3 (GND), U1.38 (GND), U1.8 (GND), U2.8 (GND), U3.8 (GND), U4.8 (GND), U5.8 (GND), U6.7 (GND), U7.13 (GND), USIPO0.13 (~{OE}), USIPO0.8 (GND), USIPO1.13 (~{OE}), USIPO1.8 (GND), USIPO2.13 (~{OE}), USIPO2.8 (GND)
- net at LED6.2 (DOUT): now also LED7.3 (DIN); no longer LED11.3 (DIN)
- net at LED1.2 (DOUT): now also LED2.3 (DIN); no longer LED6.3 (DIN)
- net at LED2.2 (DOUT): now also LED3.3 (DIN); no longer LED7.3 (DIN)
- net at LED31.2 (DOUT): no longer LED2.3 (DIN)
- net at LED22.3 (DIN): now also LED21.2 (DOUT); no longer LED17.2 (DOUT)
- net at LED12.2 (DOUT): now also LED13.3 (DIN); no longer LED17.3 (DIN)
- net at LED23.3 (DIN): now also LED22.2 (DOUT); no longer LED18.2 (DOUT)
- net at LED18.3 (DIN): now also LED17.2 (DOUT); no longer LED13.2 (DOUT)
- net at LED30.2 (DOUT): now also LED31.3 (DIN)
- net at LED28.3 (DIN): now also LED27.2 (DOUT); no longer LED23.2 (DOUT)
- net at LED29.2 (DOUT): now also LED30.3 (DIN)
- net at LED29.3 (DIN): now also LED28.2 (DOUT); no longer LED24.2 (DOUT)
- net at LED26.3 (DIN): now also LED25.2 (DOUT); no longer LED21.2 (DOUT)
- net at LED21.3 (DIN): now also LED20.2 (DOUT); no longer LED16.2 (DOUT)
- net at LED4.3 (DIN): now also LED3.2 (DOUT)
- net at LED26.2 (DOUT): now also LED27.3 (DIN); no longer LED31.3 (DIN)
- net at LED25.3 (DIN): now also LED24.2 (DOUT); no longer LED20.2 (DOUT)
- net at LED15.3 (DIN): now also LED14.2 (DOUT); no longer LED10.2 (DOUT)
- net at LED10.3 (DIN): now also LED9.2 (DOUT); no longer LED5.2 (DOUT)
- net at LED19.3 (DIN): now also LED18.2 (DOUT); no longer LED14.2 (DOUT)
- net at LED14.3 (DIN): now also LED13.2 (DOUT); no longer LED9.2 (DOUT)
- net at LED20.3 (DIN): now also LED19.2 (DOUT); no longer LED15.2 (DOUT)
- net at LED12.3 (DIN): now also LED11.2 (DOUT); no longer LED7.2 (DOUT)
- net at LED8.2 (DOUT): now also LED9.3 (DIN); no longer LED13.3 (DIN)
- net at LED8.3 (DIN): now also LED7.2 (DOUT); no longer LED3.2 (DOUT)
- net at LED24.3 (DIN): now also LED23.2 (DOUT); no longer LED19.2 (DOUT)
- net at LED4.2 (DOUT): now also LED5.3 (DIN); no longer LED9.3 (DIN)
- net at LED16.3 (DIN): now also LED15.2 (DOUT); no longer LED11.2 (DOUT)
- net WS2812: no longer names the net of LED1.3 (DIN)
- net WS2812: now also LED0.2 (DOUT)
- new net: R2.2, SW2.2, U2.3 (D)
- new net: R20.2, SW20.2, U4.5 (F)
- new net: R16.2, SW16.2, U4.1 (B)
- new net: R18.2, SW18.2, U4.3 (D)
- new net: R5.2, SW5.2, U2.6 (G)
- new net: R11.2, SW11.2, U3.15 (A)
- new net: R22.2, SW22.2, U4.7 (H)
- new net: R13.2, SW13.2
- new net: R9.2, SW9.2, U3.2 (C)
- new net: LED16.2 (DOUT), LED17.3 (DIN)
- new net: R31.2, SW31.2, U5.15 (A)
- new net: R6.2, SW6.2, U2.15 (A)
- new net: R3.2, SW3.2, U2.4 (E)
- new net: USIPO0.9 (QH'), USIPO1.14 (SER)
- new net: USIPO1.9 (QH'), USIPO2.14 (SER)
- new net: R14.2, SW14.2
- new net: R25.2, SW25.2, U5.2 (C)
- new net: R19.2, SW19.2, U4.4 (E)
- new net: R7.2, SW7.2, U2.7 (H)
- new net: R24.2, SW24.2, U5.1 (B)
- new net: R26.2, SW26.2, U5.3 (D)
- new net: R10.2, SW10.2, U3.1 (B)
- new net: U3.14 (SER_{IN}), U4.9 (SER_{OUT})
- new net: R8.2, SW8.2, U3.3 (D)
- new net: U2.14 (SER_{IN}), U3.9 (SER_{OUT})
- new net: U4.14 (SER_{IN}), U5.9 (SER_{OUT})
- new net: R23.2, SW23.2, U4.15 (A)
- new net: R17.2, SW17.2, U4.2 (C)
- new net: R21.2, SW21.2, U4.6 (G)
- new net: R4.2, SW4.2, U2.5 (F)
- new net: R1.2, SW1.2, U2.2 (C)
- new net: R30.2, SW30.2, U5.7 (H)
- new net: LED10.2 (DOUT), LED11.3 (DIN)
- new net: R12.2, SW12.2
- new net: R28.2, SW28.2, U5.5 (F)
- new net: R27.2, SW27.2, U5.4 (E)
- new net: R29.2, SW29.2, U5.6 (G)
- new net: R0.2, SW0.2, U2.1 (B)
- new net: R15.2, SW15.2
- new net: LED5.2 (DOUT), LED6.3 (DIN)
- new net 9163_CS: U6.6 (CS), USIPO0.3 (QD)
- new net 9163_RST: U6.5 (RST), USIPO0.4 (QE)
- new net 91874_CS: J1.7 (Pin_7), USIPO0.1 (QB)
- new net 91874_RST: J1.11 (Pin_11), USIPO0.2 (QC)
- new net 9341_CS: U7.12 (CS), USIPO0.5 (QF)
- new net 9341_IRQ: U7.1 (IRQ)
- new net 9341_RST: U7.11 (RST), USIPO0.6 (QG)
- new net 9341_TOUCH_CS: U7.4 (CS)
- new net MISO: U1.6 (GPIO4), U7.2 (MISO)
- new net MOSI: J1.6 (Pin_6), U1.5 (GPIO3), U6.3 (MOSI), U7.3 (MOSI), U7.9 (MOSI)
- new net PISO_CS: U1.19 (GPIO14), U2.10 (OE), U3.10 (OE), U4.10 (OE), U5.10 (OE)
- new net PISO_LATCH: U1.20 (GPIO15), U2.12 (LATCH), U3.12 (LATCH), U4.12 (LATCH), U5.12 (LATCH)
- new net REGISTER_MISO: U1.16 (GPIO12), U2.9 (SER_{OUT})
- new net REGISTER_MOSI: U1.15 (GPIO11), USIPO0.14 (SER)
- new net REGISTER_SCK: U1.14 (GPIO10), U2.11 (CLK), U3.11 (CLK), U4.11 (CLK), U5.11 (CLK), USIPO0.11 (SRCLK), USIPO1.11 (SRCLK), USIPO2.11 (SRCLK)
- new net RGB_DATA: LED0.3 (DIN), U1.1 (GPIO0)
- new net SCK: J1.4 (Pin_4), U1.4 (GPIO2), U6.2 (SCK), U7.5 (SCK), U7.8 (SCK)
- new net SCREEN_DC: J1.8 (Pin_8), U6.4 (DC), U7.10 (DC), USIPO0.15 (QA)
- new net SIPO_CS: U1.17 (GPIO13), USIPO0.12 (RCLK), USIPO1.12 (RCLK), USIPO2.12 (RCLK)
- no-connect marks 2 -> 7
Other:
- note added: "IL91874"
- note added: "LED Matrix"
- note added: "MCU"
- note added: "PISO - Key "matrix""
- note added: "SIPO - Control screens"
- note added: "Screens"
- title: (none) -> Access Keyboard

Commit message: Matrix wired
Parts:
- removed LED29, LED30, LED31: MX_SK6812MINI-E, marbastlib-mx:LED_MX_6028R, symbol marbastlib-mx:MX_SK6812MINI-E
- removed R29, R30, R31: R_Small, Resistor_SMD:R_1206_3216Metric_Pad1.30x1.75mm_HandSolder, symbol Device:R_Small
- removed SW29, SW30, SW31: MX_SW, marbastlib-mx:SW_MX_1u, symbol marbastlib-mx:MX_SW_HS
- added UROW4: MC74HC589ADR2G, Package_SO:SO-16_3.9x9.9mm_P1.27mm, symbol my_components:MC74HC589ADR2G
- renumbered U2 to UROW1, U3 to UROW2, U4 to UROW3, U5 to UROW5
Connections:
- net +3V3: now also UROW4.16 (VCC); no longer SW16.1, SW17.1
- net GND: now also UROW1.15 (A), UROW1.7 (H), UROW2.15 (A), UROW2.7 (H), UROW3.15 (A), UROW3.7 (H), UROW5.14 (SER_{IN}), UROW5.15 (A), UROW5.6 (G), UROW5.7 (H), UROW4.15 (A), UROW4.7 (H), UROW4.8 (GND)
- net PISO_CS: now also UROW4.10 (OE)
- net PISO_LATCH: now also UROW1.13 (SER/PAR), UROW2.13 (SER/PAR), UROW3.13 (SER/PAR), UROW5.13 (SER/PAR), UROW4.12 (LATCH), UROW4.13 (SER/PAR)
- net REGISTER_SCK: now also UROW4.11 (CLK)
- net at R20.2, SW20.2: now also UROW4.3 (D); no longer UROW3.5 (F)
- net at R16.2, SW16.2: now also UROW3.5 (F); no longer UROW3.1 (B)
- net at R18.2, SW18.2: now also UROW4.1 (B); no longer UROW3.3 (D)
- net RGB7_OUT: now reaches LED7.2 (DOUT), LED8.3 (DIN)
- net at R11.2, SW11.2: now also UROW2.6 (G); no longer UROW2.15 (A)
- net at R22.2, SW22.2: now also UROW4.5 (F); no longer UROW3.7 (H)
- net at R13.2, SW13.2: now also UROW3.2 (C)
- net at R9.2, SW9.2: now also UROW2.4 (E); no longer UROW2.2 (C)
- net RGB15_OUT: now reaches LED15.2 (DOUT), LED16.3 (DIN)
- net at R6.2, SW6.2: now also UROW2.1 (B); no longer UROW1.15 (A)
- net at R14.2, SW14.2: now also UROW3.3 (D)
- net at R19.2, SW19.2: now also UROW4.2 (C); no longer UROW3.4 (E)
- net at R7.2, SW7.2: now also UROW2.2 (C); no longer UROW1.7 (H)
- net at R10.2, SW10.2: now also UROW2.5 (F); no longer UROW2.1 (B)
- net ROW3_OUT: now reaches UROW2.14 (SER_{IN}), UROW3.9 (SER_{OUT})
- net ROW2_OUT: now reaches UROW1.14 (SER_{IN}), UROW2.9 (SER_{OUT})
- net ROW4_OUT: now reaches UROW3.14 (SER_{IN})
- net ROW4_OUT: now also UROW4.9 (SER_{OUT}); no longer UROW5.9 (SER_{OUT})
- net at R23.2, SW23.2: now also UROW4.6 (G); no longer UROW3.15 (A)
- net at R17.2, SW17.2: now also UROW3.6 (G); no longer UROW3.2 (C)
- net at R21.2, SW21.2: now also UROW4.4 (E); no longer UROW3.6 (G)
- net RGB23_OUT: now reaches LED23.2 (DOUT), LED24.3 (DIN)
- net at R12.2, SW12.2: now also UROW3.1 (B)
- net at R15.2, SW15.2: now also UROW3.4 (E)
- new net: SW16.1, SW17.1
- new net ROW5_OUT: UROW4.14 (SER_{IN}), UROW5.9 (SER_{OUT})
Other:
- moved on the sheet: R0, R1, R10, R11, R12, R13, R14, R15, R16, R17, R18, R19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
