File: hardware/kicad/kicad.kicad_sch (KiCad schematic)
At the start: 99 parts, among them J1 Conn_01x13_Female, SW0 MX_SW, SW1 MX_SW, SW10 MX_SW, SW11 MX_SW, SW12 MX_SW, SW13 MX_SW, SW14 MX_SW, SW15 MX_SW, SW16 MX_SW, SW17 MX_SW, SW18 MX_SW, SW19 MX_SW, SW2 MX_SW, SW20 MX_SW, SW21 MX_SW, SW22 MX_SW, SW23 MX_SW, SW24 MX_SW, SW25 MX_SW, SW26 MX_SW, SW27 MX_SW, SW28 MX_SW, SW3 MX_SW, SW4 MX_SW, SW5 MX_SW, SW6 MX_SW, SW7 MX_SW, SW8 MX_SW, SW9 MX_SW, U1 Pico, U6 ILI9163, U7 ILI9341_TS

Commit message: Second half added
Parts:
- removed J1: Conn_01x13_Female, Connector_PinHeader_1.00mm:PinHeader_1x13_P1.00mm_Vertical, symbol Connector:Conn_01x13_Female
- removed U6: ILI9163, my_components:ILI9163, symbol my_components:ILI9163
- removed U7: ILI9341_TS, my_components:ILI9341_TS, symbol my_components:ILI9341_TS
- added J1, J2: AudioJack4, Connector_Audio:Jack_3.5mm_KoreanHropartsElec_PJ-320D-4A_Horizontal, symbol Connector:AudioJack4
- added LED29, LED30, LED31, LED32, LED33, LED34, LED35, LED36, LED37, LED38, LED39, LED40, LED41, LED42, LED43, LED44, LED45, LED46, LED47, LED48, LED49, LED50, LED51, LED52, LED53, LED54, LED55, LED56, LED57: MX_SK6812MINI-E, marbastlib-mx:LED_MX_6028R, symbol marbastlib-mx:MX_SK6812MINI-E
- added Q1, Q2: 2N7002, Package_TO_SOT_SMD:SOT-23, symbol Transistor_FET:2N7002
- added R29, R30, R31, R32, R33, R34, R35, R36, R37, R38, R39, R40, R41, R42, R43, R44, R45, R46, R47, R48, R49, R50, R51, R52, R53, R54, R55, R56, R57, R58, R59: R_Small, Resistor_SMD:R_1206_3216Metric_Pad1.30x1.75mm_HandSolder, symbol Device:R_Small
- added SW29, SW30, SW31, SW32, SW33, SW34, SW35, SW36, SW37, SW38, SW39, SW40, SW41, SW42, SW43, SW44, SW45, SW46, SW47, SW48, SW49, SW50, SW51, SW52, SW53, SW54, SW55, SW56, SW57: MX_SW, marbastlib-mx:SW_MX_1u, symbol marbastlib-mx:MX_SW_HS
- added U2: Pico, MCU_RaspberryPi_and_Boards:RPi_Pico_SMD_TH, symbol MCU_RaspberryPi_and_Boards:Pico
- added U3: ILI9163, my_components:ILI9163, symbol my_components:ILI9163
- added U4: ILI9341_TS, my_components:ILI9341_TS, symbol my_components:ILI9341_TS
- added U5: IL91874, my_components:IL91874, symbol my_components:IL91874
- added UROW10, UROW6, UROW7, UROW8, UROW9: MC74HC589ADR2G, Package_SO:SO-16_3.9x9.9mm_P1.27mm, symbol my_components:MC74HC589ADR2G
- added USIPO3: 74HC595, Package_SO:SO-16_3.9x9.9mm_P1.27mm, symbol 74xx:74HC595
Connections:
- net +3V3: now also SW16.1, SW17.1, J1.S, J2.S, LED29.1 (VDD), LED30.1 (VDD), LED31.1 (VDD), LED32.1 (VDD), LED33.1 (VDD), LED34.1 (VDD), LED35.1 (VDD), LED36.1 (VDD), LED37.1 (VDD), LED38.1 (VDD), LED39.1 (VDD), LED40.1 (VDD), LED41.1 (VDD), LED42.1 (VDD), LED43.1 (VDD), LED44.1 (VDD), LED45.1 (VDD), LED46.1 (VDD), LED47.1 (VDD), LED48.1 (VDD), LED49.1 (VDD), LED50.1 (VDD), LED51.1 (VDD), LED52.1 (VDD), LED53.1 (VDD), LED54.1 (VDD), LED55.1 (VDD), LED56.1 (VDD), LED57.1 (VDD), R29.1, R59.1, SW29.1, SW30.1, SW31.1, SW32.1, SW33.1, SW34.1, SW35.1, SW36.1, SW37.1, SW38.1, SW39.1, SW40.1, SW41.1, SW42.1, SW43.1, SW44.1, SW45.1, SW46.1, SW47.1, SW48.1, SW49.1, SW50.1, SW51.1, SW52.1, SW53.1, SW54.1, SW55.1, SW56.1, SW57.1, U2.36 (3V3), U3.1 (LED), U3.8 (VCC), U4.14 (VCC), U4.7 (LED), U5.1 (V_{IN}), UROW10.16 (VCC), UROW6.16 (VCC), UROW7.16 (VCC), UROW8.16 (VCC), UROW9.16 (VCC), USIPO3.10 (~{SRCLR}), USIPO3.16 (VCC)
- net 9163_CS: now also USIPO2.1 (QB), U3.6 (CS); no longer USIPO0.3 (QD)
- net 9163_RST: now also USIPO2.2 (QC), U3.5 (RST); no longer USIPO0.4 (QE)
- net 91874_CS: now also U5.7 (ECS)
- net 91874_RST: now also U5.11 (RST)
- net 9341_CS: now also USIPO2.3 (QD), U4.12 (CS); no longer USIPO0.5 (QF)
- net 9341_IRQ: now also U4.1 (IRQ)
- net 9341_RST: now also USIPO2.4 (QE), U4.11 (RST); no longer USIPO0.6 (QG)
- net 9341_TOUCH_CS: now also U4.4 (CS)
- net GND: now also J1.T, J2.T, LED29.4 (VSS), LED30.4 (VSS), LED31.4 (VSS), LED32.4 (VSS), LED33.4 (VSS), LED34.4 (VSS), LED35.4 (VSS), LED36.4 (VSS), LED37.4 (VSS), LED38.4 (VSS), LED39.4 (VSS), LED40.4 (VSS), LED41.4 (VSS), LED42.4 (VSS), LED43.4 (VSS), LED44.4 (VSS), LED45.4 (VSS), LED46.4 (VSS), LED47.4 (VSS), LED48.4 (VSS), LED49.4 (VSS), LED50.4 (VSS), LED51.4 (VSS), LED52.4 (VSS), LED53.4 (VSS), LED54.4 (VSS), LED55.4 (VSS), LED56.4 (VSS), LED57.4 (VSS), Q1.2 (S), Q2.2 (S), R30.1, R31.1, R32.1, R33.1, R34.1, R35.1, R36.1, R37.1, R38.1, R39.1, R40.1, R41.1, R42.1, R43.1, R44.1, R45.1, R46.1, R47.1, R48.1, R49.1, R50.1, R51.1, R52.1, R53.1, R54.1, R55.1, R56.1, R57.1, R58.1, U2.13 (GND), U2.18 (GND), U2.23 (GND), U2.28 (GND), U2.3 (GND), U2.38 (GND), U2.8 (GND), U3.7 (GND), U4.13 (GND), U5.3 (GND), UROW10.14 (SER_{IN}), UROW10.15 (A), UROW10.6 (G), UROW10.7 (H), UROW10.8 (GND), UROW6.15 (A), UROW6.7 (H), UROW6.8 (GND), UROW7.15 (A), UROW7.7 (H), UROW7.8 (GND), UROW8.15 (A), UROW8.7 (H), UROW8.8 (GND), UROW9.15 (A), UROW9.7 (H), UROW9.8 (GND), USIPO3.13 (~{OE}), USIPO3.8 (GND)
- net REGISTER_MISO: now also U2.16 (GPIO12); no longer U1.16 (GPIO12), UROW1.9 (SER_{OUT})
- net REGISTER_MOSI: now also U2.15 (GPIO11); no longer U1.15 (GPIO11), USIPO0.14 (SER)
- net at USIPO1.9 (QH'): no longer USIPO2.14 (SER)
- net SCREEN_DC_R: now reaches USIPO2.15 (QA)
- net SCREEN_DC_R: now also U3.4 (DC), U4.10 (DC)
- net at USIPO2.9 (QH'): now also USIPO3.14 (SER)
- net MISO renamed MISO_L
- net MOSI renamed MOSI_L
- net PISO_CS renamed PISO_CS_L
- net PISO_CS_L: now also USIPO0.12 (RCLK), USIPO1.12 (RCLK), Q1.1 (G)
- net PISO_LATCH renamed PISO_LATCH_L
- net PISO_LATCH_L: now also Q1.3 (D), R29.2; no longer U1.20 (GPIO15)
- net REGISTER_SCK renamed REGISTER_SCK_L
- net REGISTER_SCK_L: no longer USIPO2.11 (SRCLK)
- net RGB15_OUT renamed RGB15_OUT_L
- net RGB23_OUT renamed RGB23_OUT_L
- net RGB7_OUT renamed RGB7_OUT_L
- net RGB_DATA renamed RGB_DATA_L
- net ROW2_OUT renamed ROW2_OUT_L
- net ROW3_OUT renamed ROW3_OUT_L
- net ROW4_OUT renamed ROW4_OUT_L
- net ROW5_OUT renamed ROW5_OUT_L
- net SCK renamed SCK_L
- net SCREEN_DC renamed SCREEN_DC_L
- net SCREEN_DC_L: now also U5.8 (DC)
- removed net SIPO_CS: U1.17 (GPIO13), USIPO0.12 (RCLK), USIPO1.12 (RCLK), USIPO2.12 (RCLK)
- new net: LED29.2 (DOUT), LED30.3 (DIN)
- new net: R40.2, SW39.2, UROW7.2 (C)
- new net: LED35.2 (DOUT), LED36.3 (DIN)
- new net: LED34.2 (DOUT), LED35.3 (DIN)
- new net: R44.2, SW43.2, UROW8.4 (E)
- new net: LED54.2 (DOUT), LED55.3 (DIN)
- new net: LED53.2 (DOUT), LED54.3 (DIN)
- new net: LED41.2 (DOUT), LED42.3 (DIN)
- new net: LED40.2 (DOUT), LED41.3 (DIN)
- new net: R41.2, SW40.2, UROW7.1 (B)
- new net: R39.2, SW38.2, UROW7.3 (D)
- new net: R38.2, SW37.2, UROW7.4 (E)
- new net: R37.2, SW36.2, UROW7.5 (F)
- new net: R36.2, SW35.2, UROW7.6 (G)
- new net: LED31.2 (DOUT), LED32.3 (DIN)
- new net: LED30.2 (DOUT), LED31.3 (DIN)
- new net: LED39.2 (DOUT), LED40.3 (DIN)
- new net: R52.2, SW51.2, UROW9.2 (C)
- new net: R58.2, SW57.2, UROW10.1 (B)
- new net: R55.2, SW54.2, UROW10.4 (E)
- new net: LED56.2 (DOUT), LED57.3 (DIN)
- new net: R45.2, SW44.2, UROW8.3 (D)
- new net: R35.2, SW34.2, UROW6.1 (B)
- new net: R53.2, SW52.2, UROW9.1 (B)
- new net: R31.2, SW30.2, UROW6.5 (F)
- new net: LED43.2 (DOUT), LED44.3 (DIN)
- new net: LED42.2 (DOUT), LED43.3 (DIN)
- new net: R34.2, SW33.2, UROW6.2 (C)
- new net: LED46.2 (DOUT), LED47.3 (DIN)
- new net: LED45.2 (DOUT), LED46.3 (DIN)
- new net: R42.2, SW41.2, UROW8.6 (G)
- new net: R48.2, SW47.2, UROW9.6 (G)
- new net: LED49.2 (DOUT), LED50.3 (DIN)
- new net: LED48.2 (DOUT), LED49.3 (DIN)
- new net: R51.2, SW50.2, UROW9.3 (D)
- new net: LED55.2 (DOUT), LED56.3 (DIN)
- new net: LED37.2 (DOUT), LED38.3 (DIN)
- new net: R47.2, SW46.2, UROW8.1 (B)
- new net: LED38.2 (DOUT), LED39.3 (DIN)
- new net: R46.2, SW45.2, UROW8.2 (C)
- new net: LED47.2 (DOUT), LED48.3 (DIN)
- new net: R43.2, SW42.2, UROW8.5 (F)
- new net: LED50.2 (DOUT), LED51.3 (DIN)
- new net: R54.2, SW53.2, UROW10.5 (F)
- new net: LED33.2 (DOUT), LED34.3 (DIN)
- new net: R56.2, SW55.2, UROW10.3 (D)
- new net: R30.2, SW29.2, UROW6.6 (G)
- new net: LED32.2 (DOUT), LED33.3 (DIN)
- new net: LED51.2 (DOUT), LED52.3 (DIN)
- new net: R57.2, SW56.2, UROW10.2 (C)
- new net: R32.2, SW31.2, UROW6.4 (E)
- new net: R50.2, SW49.2, UROW9.4 (E)
- new net: R33.2, SW32.2, UROW6.3 (D)
- new net: R49.2, SW48.2, UROW9.5 (F)
- new net MISO_R: U2.6 (GPIO4), U4.2 (MISO)
- new net MOSI_R: U2.5 (GPIO3), U3.3 (MOSI), U4.3 (MOSI), U4.9 (MOSI), U5.6 (MOSI)
- new net PISO_CS_R: Q2.1 (G), U2.19 (GPIO14), UROW10.10 (OE), UROW6.10 (OE), UROW7.10 (OE), UROW8.10 (OE), UROW9.10 (OE)
- new net PISO_LATCH_R: Q2.3 (D), R59.2, UROW10.12 (LATCH), UROW10.13 (SER/PAR), UROW6.12 (LATCH), UROW6.13 (SER/PAR), UROW7.12 (LATCH), UROW7.13 (SER/PAR), UROW8.12 (LATCH), UROW8.13 (SER/PAR), UROW9.12 (LATCH), UROW9.13 (SER/PAR)
- new net REGISTER_MISO_L: U1.16 (GPIO12), UROW1.9 (SER_{OUT})
- new net REGISTER_MISO_R: UROW6.9 (SER_{OUT})
- new net REGISTER_MOSI_L: U1.15 (GPIO11), USIPO0.14 (SER)
- new net REGISTER_MOSI_R: USIPO2.14 (SER)
- new net REGISTER_SCK_R: U2.14 (GPIO10), UROW10.11 (CLK), UROW6.11 (CLK), UROW7.11 (CLK), UROW8.11 (CLK), UROW9.11 (CLK), USIPO2.11 (SRCLK), USIPO3.11 (SRCLK)
- new net RGB15_OUT_R: LED44.2 (DOUT), LED45.3 (DIN)
- new net RGB23_OUT_R: LED52.2 (DOUT), LED53.3 (DIN)
- new net RGB7_OUT_R: LED36.2 (DOUT), LED37.3 (DIN)
- new net RGB_DATA_R: LED29.3 (DIN), U2.1 (GPIO0)
- new net ROW2_OUT_R: UROW6.14 (SER_{IN}), UROW7.9 (SER_{OUT})
- new net ROW3_OUT_R: UROW7.14 (SER_{IN}), UROW8.9 (SER_{OUT})
- new net ROW4_OUT_R: UROW8.14 (SER_{IN}), UROW9.9 (SER_{OUT})
- new net ROW5_OUT_R: UROW10.9 (SER_{OUT}), UROW9.14 (SER_{IN})
- new net SCK_R: U2.4 (GPIO2), U3.2 (SCK), U4.5 (SCK), U4.8 (SCK), U5.4 (SCK)
- new net SIPO_CS_L: U1.17 (GPIO13)
- new net SIPO_CS_R: U2.17 (GPIO13), USIPO2.12 (RCLK), USIPO3.12 (RCLK)
Other:
- note added: "LEFT"
- note added: "RIGHT"
- moved on the sheet: LED0, LED1, LED10, LED11, LED12, LED13, LED14, LED15, LED16, LED17, LED18, LED19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
