File: hardware/kicad/kicad.kicad_sch (KiCad schematic)
At the start: 211 parts, among them J1 AudioJack4, J2 AudioJack4, Q1 2N7002, Q2 2N7002, SW0 MX_SW, SW1 MX_SW, SW10 MX_SW, SW11 MX_SW, SW12 MX_SW, SW13 MX_SW, SW14 MX_SW, SW15 MX_SW, SW16 MX_SW, SW17 MX_SW, SW18 MX_SW, SW19 MX_SW, SW2 MX_SW, SW20 MX_SW, SW21 MX_SW, SW22 MX_SW, SW23 MX_SW, SW24 MX_SW, SW25 MX_SW, SW26 MX_SW, SW27 MX_SW, SW28 MX_SW, SW29 MX_SW, SW3 MX_SW, SW30 MX_SW, SW31 MX_SW, SW32 MX_SW, SW33 MX_SW, SW34 MX_SW, SW35 MX_SW, SW36 MX_SW, SW37 MX_SW, SW38 MX_SW, SW39 MX_SW, SW4 MX_SW, SW40 MX_SW, SW41 MX_SW, SW42 MX_SW, SW43 MX_SW, SW44 MX_SW, SW45 MX_SW, SW46 MX_SW, SW47 MX_SW, SW48 MX_SW, SW49 MX_SW, SW5 MX_SW, SW50 MX_SW, SW51 MX_SW, SW52 MX_SW, SW53 MX_SW, SW54 MX_SW, SW55 MX_SW, SW56 MX_SW, SW57 MX_SW, SW6 MX_SW, SW7 MX_SW, SW8 MX_SW, SW9 MX_SW, U1 Pico, U2 Pico, U3 ILI9163, U4 ILI9341_TS, U5 IL91874

Commit message: Done?
Parts:
- added J10, J9: Conn_02x02_Top_Bottom, Connector_PinHeader_2.54mm:PinHeader_2x02_P2.54mm_Vertical, symbol Connector_Generic:Conn_02x02_Top_Bottom
- added J3, J4, J6, J8: Conn_02x03_Top_Bottom, Connector_PinHeader_2.54mm:PinHeader_2x03_P2.54mm_Vertical, symbol Connector_Generic:Conn_02x03_Top_Bottom
- added J5, J7: Conn_01x17_Female, Connector_PinHeader_2.54mm:PinHeader_1x17_P2.54mm_Vertical, symbol Connector:Conn_01x17_Female
- U3: footprint my_components:ILI9163 -> Connector_PinHeader_2.54mm:PinHeader_1x08_P2.54mm_Vertical
- U4: footprint my_components:ILI9341_TS -> Connector_PinHeader_2.54mm:PinHeader_1x14_P2.54mm_Vertical
- U5: footprint my_components:IL91874 -> Connector_PinHeader_2.54mm:PinHeader_1x13_P2.54mm_Vertical
- gave numbers to parts that had none: 2
Connections:
- net +3V3: now also J6.1 (Pin_1), J6.2 (Pin_2), J6.3 (Pin_3), J6.4 (Pin_4), J6.5 (Pin_5), J6.6 (Pin_6), J8.1 (Pin_1), J8.2 (Pin_2), J8.3 (Pin_3), J8.4 (Pin_4), J8.5 (Pin_5), J8.6 (Pin_6); no longer J1.S, J2.S
- net 9341_IRQ: now also UROW10.15 (A)
- net 9341_TOUCH_CS: now also USIPO2.15 (QA)
- net GND: now also J3.1 (Pin_1), J3.2 (Pin_2), J3.3 (Pin_3), J3.4 (Pin_4), J3.5 (Pin_5), J3.6 (Pin_6), J4.1 (Pin_1), J4.2 (Pin_2), J4.3 (Pin_3), J4.4 (Pin_4), J4.5 (Pin_5), J4.6 (Pin_6); no longer UROW10.15 (A), UROW10.6 (G)
- net GPIO7_R: now reaches U2.10 (GPIO7)
- net GPIO7_R: now also J7.13 (Pin_13)
- net GPIO8_R: now reaches U2.11 (GPIO8)
- net GPIO8_R: now also J7.14 (Pin_14)
- net GPIO9_R: now reaches U2.12 (GPIO9)
- net GPIO9_R: now also J7.15 (Pin_15)
- net GPIO14_R: now reaches U2.19 (GPIO14)
- net GPIO14_R: now also J7.16 (Pin_16)
- net GPIO15_R: now reaches U2.20 (GPIO15)
- net GPIO15_R: now also J7.17 (Pin_17)
- net GPIO16_R: now reaches U2.21 (GPIO16)
- net GPIO16_R: now also J7.10 (Pin_10)
- net GPIO17_R: now reaches U2.22 (GPIO17)
- net GPIO17_R: now also J7.9 (Pin_9)
- net GPIO18_R: now reaches U2.24 (GPIO18)
- net GPIO18_R: now also J7.8 (Pin_8)
- net GPIO19_R: now reaches U2.25 (GPIO19)
- net GPIO19_R: now also J7.7 (Pin_7)
- net GPIO20_R: now reaches U2.26 (GPIO20)
- net GPIO20_R: now also J7.6 (Pin_6)
- net GPIO21_R: now reaches U2.27 (GPIO21)
- net GPIO21_R: now also J7.5 (Pin_5)
- net GPIO22_R: now reaches U2.29 (GPIO22)
- net GPIO22_R: now also J7.4 (Pin_4)
- net GPIO23_R: now reaches U2.31 (GPIO26_ADC0)
- net GPIO23_R: now also J7.3 (Pin_3)
- net GPIO24_R: now reaches U2.32 (GPIO27_ADC1)
- net GPIO24_R: now also J7.2 (Pin_2)
- net GPIO28_R: now reaches U2.34 (GPIO28_ADC2)
- net GPIO28_R: now also J7.1 (Pin_1)
- net VSYS_R: now reaches U2.39 (VSYS)
- net VSYS_R: now also J2.S, J10.1 (Pin_1), J10.2 (Pin_2), J10.3 (Pin_3), J10.4 (Pin_4)
- net GPIO5_R: now reaches U2.7 (GPIO5)
- net GPIO5_R: now also J7.11 (Pin_11)
- net GPIO6_R: now reaches U2.9 (GPIO6)
- net GPIO6_R: now also J7.12 (Pin_12)
- net GPIO7_L: now reaches U1.10 (GPIO7)
- net GPIO7_L: now also J5.13 (Pin_13)
- net GPIO8_L: now reaches U1.11 (GPIO8)
- net GPIO8_L: now also J5.14 (Pin_14)
- net GPIO9_L: now reaches U1.12 (GPIO9)
- net GPIO9_L: now also J5.15 (Pin_15)
- net GPIO14_L: now reaches U1.19 (GPIO14)
- net GPIO14_L: now also J5.16 (Pin_16)
- net GPIO15_L: now reaches U1.20 (GPIO15)
- net GPIO15_L: now also J5.17 (Pin_17)
- net GPIO16_L: now reaches U1.21 (GPIO16)
- net GPIO16_L: now also J5.10 (Pin_10)
- net GPIO17_L: now reaches U1.22 (GPIO17)
- net GPIO17_L: now also J5.9 (Pin_9)
- net GPIO18_L: now reaches U1.24 (GPIO18)
- net GPIO18_L: now also J5.8 (Pin_8)
- net GPIO19_L: now reaches U1.25 (GPIO19)
- net GPIO19_L: now also J5.7 (Pin_7)
- net GPIO20_L: now reaches U1.26 (GPIO20)
- net GPIO20_L: now also J5.6 (Pin_6)
- net GPIO21_L: now reaches U1.27 (GPIO21)
- net GPIO21_L: now also J5.5 (Pin_5)
- net GPIO22_L: now reaches U1.29 (GPIO22)
- net GPIO22_L: now also J5.4 (Pin_4)
- net GPIO23_L: now reaches U1.31 (GPIO26_ADC0)
- net GPIO23_L: now also J5.3 (Pin_3)
- net GPIO24_L: now reaches U1.32 (GPIO27_ADC1)
- net GPIO24_L: now also J5.2 (Pin_2)
- net GPIO28_L: now reaches U1.34 (GPIO28_ADC2)
- net GPIO28_L: now also J5.1 (Pin_1)
- net VSYS_L: now reaches U1.39 (VSYS)
- net VSYS_L: now also J1.S, J9.1 (Pin_1), J9.2 (Pin_2), J9.3 (Pin_3), J9.4 (Pin_4)
- net GPIO5_L: now reaches U1.7 (GPIO5)
- net GPIO5_L: now also J5.11 (Pin_11)
- net GPIO6_L: now reaches U1.9 (GPIO6)
- net GPIO6_L: now also J5.12 (Pin_12)
Other:
- note added: "GPIO Breakout"
- note added: "Inverter"
- note added: "Mounting holes"
- note added: "Power Breakout"
- note added: "Split comms"
- moved on the sheet: H1, H10, H11, H12, H2, H3, H4, H5, H6, H7, H8, H9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

Commit message: Add capacitors, fix vias in pads and add SIPO connector
Parts:
- removed J5, J7: Conn_01x17_Female, Connector_PinHeader_2.54mm:PinHeader_1x17_P2.54mm_Vertical, symbol Connector:Conn_01x17_Female
- added C1, C10, C11, C12, C13, C14, C15, C16, C17, C18, C19, C2, C20, C21, C22, C23, C24, C25, C26, C27, C28, C29, C3, C30, C31, C32, C33, C34, C35, C36, C37, C38, C39, C4, C40, C41, C42, C43, C44, C45, C46, C47, C48, C49, C5, C50, C51, C52, C53, C54, C55, C56, C57, C58, C59, C6, C60, C61, C62, C63, C64, C65, C66, C67, C68, C69, C7, C70, C71, C72, C8, C9: C_Small, Capacitor_SMD:C_1206_3216Metric_Pad1.33x1.80mm_HandSolder, symbol Device:C_Small
- added J11: Conn_01x10_Female, Connector_PinSocket_2.54mm:PinSocket_1x10_P2.54mm_Vertical, symbol Connector:Conn_01x10_Female
- added J5, J7: Conn_01x16_Female, Connector_PinSocket_2.54mm:PinSocket_1x16_P2.54mm_Vertical, symbol Connector:Conn_01x16_Female
- J10, J9: footprint Connector_PinHeader_2.54mm:PinHeader_2x02_P2.54mm_Vertical -> Connector_PinSocket_2.54mm:PinSocket_2x02_P2.54mm_Vertical
- J3, J4, J6, J8: footprint Connector_PinHeader_2.54mm:PinHeader_2x03_P2.54mm_Vertical -> Connector_PinSocket_2.54mm:PinSocket_2x03_P2.54mm_Vertical
- U3: footprint Connector_PinHeader_2.54mm:PinHeader_1x08_P2.54mm_Vertical -> Connector_PinSocket_2.54mm:PinSocket_1x08_P2.54mm_Vertical
- U4: footprint Connector_PinHeader_2.54mm:PinHeader_1x14_P2.54mm_Vertical -> Connector_PinSocket_2.54mm:PinSocket_1x14_P2.54mm_Vertical
- U5: footprint Connector_PinHeader_2.54mm:PinHeader_1x13_P2.54mm_Vertical -> Connector_PinSocket_2.54mm:PinSocket_1x13_P2.54mm_Vertical
Connections:
- net GPIO15_L is gone; now on net COMMS_L: U1.20 (GPIO15)
- net GPIO15_R is gone; now on net COMMS_R: U2.20 (GPIO15)
- net +3V3: now also C1.2, C10.2, C11.2, C12.2, C13.2, C14.2, C15.2, C16.2, C17.2, C18.2, C19.2, C2.2, C20.2, C21.2, C22.2, C23.2, C24.2, C25.2, C26.2, C27.2, C28.2, C29.2, C3.2, C30.2, C31.2, C32.2, C33.2, C34.2, C35.2, C36.2, C37.2, C38.2, C39.2, C4.2, C40.2, C41.2, C42.2, C43.2, C44.2, C45.2, C46.2, C47.2, C48.2, C49.2, C5.2, C50.2, C51.2, C52.2, C53.2, C54.2, C55.2, C56.2, C57.2, C58.2, C59.2, C6.2, C60.2, C61.2, C62.2, C63.2, C64.2, C65.2, C66.2, C67.2, C68.2, C69.2, C7.2, C70.2, C71.2, C72.2, C8.2, C9.2
- net GND: now also C1.1, C10.1, C11.1, C12.1, C13.1, C14.1, C15.1, C16.1, C17.1, C18.1, C19.1, C2.1, C20.1, C21.1, C22.1, C23.1, C24.1, C25.1, C26.1, C27.1, C28.1, C29.1, C3.1, C30.1, C31.1, C32.1, C33.1, C34.1, C35.1, C36.1, C37.1, C38.1, C39.1, C4.1, C40.1, C41.1, C42.1, C43.1, C44.1, C45.1, C46.1, C47.1, C48.1, C49.1, C5.1, C50.1, C51.1, C52.1, C53.1, C54.1, C55.1, C56.1, C57.1, C58.1, C59.1, C6.1, C60.1, C61.1, C62.1, C63.1, C64.1, C65.1, C66.1, C67.1, C68.1, C69.1, C7.1, C70.1, C71.1, C72.1, C8.1, C9.1
- net GPIO14_L: now also J5.16 (Pin_16)
- net GPIO14_R: now also J7.16 (Pin_16)
- net GPIO16_L: now also J5.10 (Pin_10)
- net GPIO16_R: now also J7.10 (Pin_10)
- net GPIO17_L: now also J5.9 (Pin_9)
- net GPIO17_R: now also J7.9 (Pin_9)
- net GPIO18_L: now also J5.8 (Pin_8)
- net GPIO18_R: now also J7.8 (Pin_8)
- net GPIO19_L: now also J5.7 (Pin_7)
- net GPIO19_R: now also J7.7 (Pin_7)
- net GPIO20_L: now also J5.6 (Pin_6)
- net GPIO20_R: now also J7.6 (Pin_6)
- net GPIO21_L: now also J5.5 (Pin_5)
- net GPIO21_R: now also J7.5 (Pin_5)
- net GPIO22_L: now also J5.4 (Pin_4)
- net GPIO22_R: now also J7.4 (Pin_4)
- net GPIO23_L: now also J5.3 (Pin_3)
- net GPIO23_R: now also J7.3 (Pin_3)
- net GPIO24_L: now also J5.2 (Pin_2)
- net GPIO24_R: now also J7.2 (Pin_2)
- net GPIO28_L: now also J5.1 (Pin_1)
- net GPIO28_R: now also J7.1 (Pin_1)
- net GPIO5_L: now also J5.11 (Pin_11)
- net GPIO5_R: now also J7.11 (Pin_11)
- net GPIO6_L: now also J5.12 (Pin_12)
- net GPIO6_R: now also J7.12 (Pin_12)
- net GPIO7_L: now also J5.13 (Pin_13)
- net GPIO7_R: now also J7.13 (Pin_13)
- net GPIO8_L: now also J5.14 (Pin_14)
- net GPIO8_R: now also J7.14 (Pin_14)
- net GPIO9_L: now also J5.15 (Pin_15)
- net GPIO9_R: now also J7.15 (Pin_15)
- net COMMS_L: now reaches J1.R1
- net SIPO_4: now reaches USIPO1.1 (QB)
- net SIPO_4: now also J11.4 (Pin_4)
- net SIPO_5: now reaches USIPO1.2 (QC)
- net SIPO_5: now also J11.5 (Pin_5)
- net SIPO_6: now reaches USIPO1.3 (QD)
- net SIPO_6: now also J11.6 (Pin_6)
- net SIPO_7: now reaches USIPO1.4 (QE)
- net SIPO_7: now also J11.7 (Pin_7)
- net SIPO_8: now reaches USIPO1.5 (QF)
- net SIPO_8: now also J11.8 (Pin_8)
- net SIPO_9: now reaches USIPO1.6 (QG)
- net SIPO_9: now also J11.9 (Pin_9)
- net SIPO_10: now reaches USIPO1.7 (QH)
- net SIPO_10: now also J11.10 (Pin_10)
- net COMMS_R: now reaches J2.R1
- net SIPO_1: now reaches USIPO0.5 (QF)
- net SIPO_1: now also J11.1 (Pin_1)
- net SIPO_2: now reaches USIPO0.6 (QG)
- net SIPO_2: now also J11.2 (Pin_2)
- net SIPO_3: now reaches USIPO0.7 (QH)
- net SIPO_3: now also J11.3 (Pin_3)
Other:
- note added: "Capacitors"
- note added: "SIPO Breakout"
- moved on the sheet: H1, H10, H11, H12, H2, H3, H4, H5, H6, H7, H8, H9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

Commit message: Fix label & Add gerbers
Connections:
- net GND: now also UROW10.6 (G)
- net PISO_CS_L: no longer USIPO0.12 (RCLK), USIPO1.12 (RCLK)
- net SIPO_CS_L: now also USIPO0.12 (RCLK), USIPO1.12 (RCLK)
- no-connect marks 5 -> 39
Changed lines of the file:
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@@
   (junction (at 87.63 173.99) (diameter 0) (color 0 0 0 0)
   )
-  (junction (at 793.75 86.36) (diameter 0) (color 0 0 0 0)
-  )
   (junction (at 519.43 127) (diameter 0) (color 0 0 0 0)
   )
@@
   (junction (at 802.64 130.81) (diameter 0) (color 0 0 0 0)
   )
-  (junction (at 774.7 71.12) (diameter 0) (color 0 0 0 0)
-  )
   (junction (at 797.56 130.81) (diameter 0) (color 0 0 0 0)
   )
@@
   (junction (at 236.22 232.41) (diameter 0) (color 0 0 0 0)
   )
+  (junction (at 793.75 86.36) (diameter 0) (color 0 0 0 0)
+  )
   (junction (at 520.7 146.05) (diameter 0) (color 0 0 0 0)
   )
@@
   (junction (at 497.84 193.04) (diameter 0) (color 0 0 0 0)
   )
+  (junction (at 774.7 86.36) (diameter 0) (color 0 0 0 0)
+  )
   (junction (at 57.15 181.61) (diameter 0) (color 0 0 0 0)
   )
@@
   (junction (at 269.24 209.55) (diameter 0) (color 0 0 0 0)
   )
-  (junction (at 774.7 86.36) (diameter 0) (color 0 0 0 0)
-  )
   (junction (at 506.73 241.3) (diameter 0) (color 0 0 0 0)
   )
@@
   (junction (at 59.69 78.74) (diameter 0) (color 0 0 0 0)
   )
+  (junction (at 774.7 71.12) (diameter 0) (color 0 0 0 0)
+  )
   (junction (at 514.35 154.94) (diameter 0) (color 0 0 0 0)
   )
@@
   (junction (at 519.43 284.48) (diameter 0) (color 0 0 0 0)
   )
+  (no_connect (at 368.3 303.53))
+  (no_connect (at 368.3 328.93))
+  (no_connect (at 463.55 308.61))
+  (no_connect (at 347.98 356.87))
   (no_connect (at 370.84 410.21))
+  (no_connect (at 367.03 520.7))
+  (no_connect (at 504.19 389.89))
+  (no_connect (at 444.5 402.59))
+  (no_connect (at 444.5 405.13))
+  (no_connect (at 504.19 400.05))
+  (no_connect (at 463.55 316.23))
+  (no_connect (at 504.19 402.59))
+  (no_connect (at 368.3 316.23))
   (no_connect (at 370.84 384.81))
+  (no_connect (at 444.5 521.97))
+  (no_connect (at 463.55 321.31))
   (no_connect (at 370.84 405.13))
+  (no_connect (at 445.77 361.95))
+  (no_connect (at 325.12 383.54))
+  (no_connect (at 504.19 405.13))
   (no_connect (at 554.99 397.51))
+  (no_connect (at 124.46 109.22))
+  (no_connect (at 504.19 410.21))
+  (no_connect (at 443.23 361.95))
+  (no_connect (at 504.19 387.35))
+  (no_connect (at 744.22 97.79))
+  (no_connect (at 265.43 383.54))
+  (no_connect (at 448.31 361.95))
+  (no_connect (at 463.55 334.01))
+  (no_connect (at 368.3 311.15))
+  (no_connect (at 463.55 326.39))
+  (no_connect (at 353.06 356.87))
+  (no_connect (at 350.52 356.87))
+  (no_connect (at 504.19 392.43))
+  (no_connect (at 325.12 406.4))
+  (no_connect (at 504.19 397.51))
+  (no_connect (at 504.19 394.97))
+  (no_connect (at 368.3 321.31))
   (no_connect (at 370.84 412.75))
   (wire (pts (xy 246.38 96.52) (xy 260.35 96.52))
@@
     (stroke (width 0) (type default) (color 0 0 0 0))
   )
-  (wire (pts (xy 774.7 71.12) (xy 793.75 71.12))
-    (stroke (width 0) (type default) (color 0 0 0 0))
-  )
   (wire (pts (xy 717.55 71.12) (xy 736.6 71.12))
     (stroke (width 0) (type default) (color 0 0 0 0))
@@
     (stroke (width 0) (type default) (color 0 0 0 0))
   )
-  (wire (pts (xy 744.22 97.79) (xy 748.03 97.79))
-    (stroke (width 0) (type default) (color 0 0 0 0))
-  )
   (wire (pts (xy 521.97 113.03) (xy 521.97 124.46))
     (stroke (width 0) (type default) (color 0 0 0 0))
@@
     (stroke (width 0) (type default) (color 0 0 0 0))
   )
+  (wire (pts (xy 774.7 71.12) (xy 793.75 71.12))
+    (stroke (width 0) (type default) (color 0 0 0 0))
+  )
   (wire (pts (xy 30.48 82.55) (xy 40.64 82.55))
     (stroke (width 0) (type default) (color 0 0 0 0))
@@
     (stroke (width 0) (type default) (color 0 0 0 0))
   )
+  (wire (pts (xy 774.7 86.36) (xy 793.75 86.36))
+    (stroke (width 0) (type default) (color 0 0 0 0))
+  )
   (wire (pts (xy 525.78 86.36) (xy 502.92 86.36))
     (stroke (width 0) (type default) (color 0 0 0 0))
@@
     (stroke (width 0) (type default) (color 0 0 0 0))
   )
-  (wire (pts (xy 774.7 86.36) (xy 793.75 86.36))
-    (stroke (width 0) (type default) (color 0 0 0 0))
-  )
   (wire (pts (xy 62.23 161.29) (xy 67.31 161.29))
     (stroke (width 0) (type default) (color 0 0 0 0))
@@
     (stroke (width 0) (type default) (color 0 0 0 0))
   )
-  (wire (pts (xy 124.46 109.22) (xy 128.27 109.22))
-    (stroke (width 0) (type default) (color 0 0 0 0))
-  )
   (wire (pts (xy 143.51 90.17) (xy 147.32 90.17))
     (stroke (width 0) (type default) (color 0 0 0 0))
@@
     )
   )
-  (global_label "PISO_CS_L" (shape input) (at 245.11 396.24 180) (fields_autoplaced)
-    (effects (font (size 1.27 1.27)) (justify right))
-    (property "Intersheet References" "${INTERSHEET_REFS}" (id 0) (at 232.8393 396.1606 0)
-      (effects (font (size 1.27 1.27)) (justify right) hide)
-    )
-  )
   (global_label "RGB23_OUT_L" (shape input) (at 33.02 109.22 180) (fields_autoplaced)
     (effects (font (size 1.27 1.27)) (justify right))
@@
     )
   )
-  (global_label "PISO_CS_L" (shape input) (at 304.8 396.24 180) (fields_autoplaced)
-    (effects (font (size 1.27 1.27)) (justify right))
-    (property "Intersheet References" "${INTERSHEET_REFS}" (id 0) (at 292.5293 396.1606 0)
-      (effects (font (size 1.27 1.27)) (justify right) hide)
-    )
-  )
   (global_label "SIPO_1" (shape input) (at 265.43 454.66 180) (fields_autoplaced)
     (effects (font (size 1.27 1.27)) (justify right))
@@
     )
   )
+  (global_label "SIPO_CS_L" (shape input) (at 245.11 396.24 180) (fields_autoplaced)
+    (effects (font (size 1.27 1.27)) (justify right))
+    (property "Intersheet References" "${INTERSHEET_REFS}" (id 0) (at 232.8393 396.1606 0)
+      (effects (font (size 1.27 1.27)) (justify right) hide)
+    )
+  )
   (global_label "ROW5_OUT_R" (shape input) (at 563.88 271.78 0) (fields_autoplaced)
     (effects (font (size 1.27 1.27)) (justify left))
@@
     )
   )
+  (global_label "SIPO_CS_L" (shape input) (at 304.8 396.24 180) (fields_autoplaced)
+    (effects (font (size 1.27 1.27)) (justify right))
+    (property "Intersheet References" "${INTERSHEET_REFS}" (id 0) (at 292.5293 396.1606 0)
+      (effects (font (size 1.27 1.27)) (justify right) hide)
+    )
+  )
   (global_label "MOSI_L" (shape input) (at 370.84 394.97 180) (fields_autoplaced)
     (effects (font (size 1.27 1.27)) (justify right))
@@
     (pin "2")
   )
+  (symbol (lib_id "power:GND") (at 538.48 271.78 270) (unit 1)
+    (in_bom yes) (on_board yes) (fields_autoplaced)
+    (property "Reference" "#PWR0253" (id 0) (at 532.13 271.78 0)
+      (effects (font (size 1.27 1.27)) hide)
+    )
+    (property "Value" "GND" (id 1) (at 534.67 271.7799 90)
+      (effects (font (size 1.27 1.27)) (justify right))
+    )
+    (property "Footprint" "" (id 2) (at 538.48 271.78 0)
+      (effects (font (size 1.27 1.27)) hide)
+    )
+    (property "Datasheet" "" (id 3) (at 538.48 271.78 0)
+      (effects (font (size 1.27 1.27)) hide)
+    )
+    (pin "1")
+  )
   (symbol (lib_id "power:GND") (at 805.18 67.31 0) (unit 1)
     (in_bom yes) (on_board yes) (fields_autoplaced)
@@
       (reference "#PWR0252") (unit 1) (value "GND") (footprint "")
     )
+    (path "/1e69ea97-f156-4858-bf36-9f511095b7d2"
+      (reference "#PWR0253") (unit 1) (value "GND") (footprint "")
+    )
     (path "/6cf076b0-4aa7-48d1-bf18-8a80f7c8ea31"

Commit message: Some progress
Other:
- note added: "Power flags"
Changed lines of the file:
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@@
     (effects (font (size 5 5) (thickness 1) bold italic) (justify left bottom))
   )
+  (text "Power flags" (at 379.73 85.09 0)
+    (effects (font (size 5 5) bold) (justify left bottom))
+  )
   (text "Capacitors\n" (at 768.35 116.84 0)
     (effects (font (size 3 3) (thickness 0.6) bold) (justify left bottom))
@@
     )
   )
+  (global_label "VSYS_L" (shape input) (at 382.27 95.25 90) (fields_autoplaced)
+    (effects (font (size 1.27 1.27)) (justify left))
+    (property "Intersheet References" "${INTERSHEET_REFS}" (id 0) (at 382.1906 86.245 90)
+      (effects (font (size 1.27 1.27)) (justify left) hide)
+    )
+  )
   (global_label "PISO_LATCH_L" (shape input) (at 316.23 125.73 0) (fields_autoplaced)
     (effects (font (size 1.27 1.27)) (justify left))
@@
     )
   )
+  (global_label "VSYS_R" (shape input) (at 419.1 96.52 90) (fields_autoplaced)
+    (effects (font (size 1.27 1.27)) (justify left))
+    (property "Intersheet References" "${INTERSHEET_REFS}" (id 0) (at 419.0206 87.2731 90)
+      (effects (font (size 1.27 1.27)) (justify left) hide)
+    )
+  )
   (global_label "ROW2_OUT_L" (shape input) (at 316.23 76.2 0) (fields_autoplaced)
     (effects (font (size 1.27 1.27)) (justify left))
@@
     (pin "4")
   )
+  (symbol (lib_id "power:GND") (at 408.94 92.71 0) (unit 1)
+    (in_bom yes) (on_board yes) (fields_autoplaced)
+    (property "Reference" "#PWR?" (id 0) (at 408.94 99.06 0)
+      (effects (font (size 1.27 1.27)) hide)
+    )
+    (property "Value" "GND" (id 1) (at 408.94 97.79 0))
+    (property "Footprint" "" (id 2) (at 408.94 92.71 0)
+      (effects (font (size 1.27 1.27)) hide)
+    )
+    (property "Datasheet" "" (id 3) (at 408.94 92.71 0)
+      (effects (font (size 1.27 1.27)) hide)
+    )
+    (pin "1")
+  )
   (symbol (lib_id "marbastlib-mx:MX_SW_HS") (at 518.16 143.51 180) (unit 1)
     (in_bom yes) (on_board yes) (fields_autoplaced)
@@
     (pin "2")
   )
+  (symbol (lib_id "power:PWR_FLAG") (at 419.1 96.52 180) (unit 1)
+    (in_bom yes) (on_board yes) (fields_autoplaced)
+    (property "Reference" "#FLG?" (id 0) (at 419.1 98.425 0)
+      (effects (font (size 1.27 1.27)) hide)
+    )
+    (property "Value" "PWR_FLAG" (id 1) (at 419.1 101.6 0))
+    (property "Footprint" "" (id 2) (at 419.1 96.52 0)
+      (effects (font (size 1.27 1.27)) hide)
+    )
+    (property "Datasheet" "~" (id 3) (at 419.1 96.52 0)
+      (effects (font (size 1.27 1.27)) hide)
+    )
+    (pin "1")
+  )
   (symbol (lib_id "Device:R_Small") (at 275.59 68.58 0) (unit 1)
     (in_bom yes) (on_board yes)
@@
     (pin "1")
   )
+  (symbol (lib_id "power:PWR_FLAG") (at 394.97 92.71 180) (unit 1)
+    (in_bom yes) (on_board yes) (fields_autoplaced)
+    (property "Reference" "#FLG0101" (id 0) (at 394.97 94.615 0)
+      (effects (font (size 1.27 1.27)) hide)
+    )
+    (property "Value" "PWR_FLAG" (id 1) (at 394.97 97.79 0))
+    (property "Footprint" "" (id 2) (at 394.97 92.71 0)
+      (effects (font (size 1.27 1.27)) hide)
+    )
+    (property "Datasheet" "~" (id 3) (at 394.97 92.71 0)
+      (effects (font (size 1.27 1.27)) hide)
+    )
+    (pin "1")
+  )
   (symbol (lib_id "power:+3V3") (at 478.79 472.44 90) (unit 1)
     (in_bom yes) (on_board yes)
@@
     (pin "1")
   )
+  (symbol (lib_id "power:+3V3") (at 394.97 92.71 0) (unit 1)
+    (in_bom yes) (on_board yes) (fields_autoplaced)
+    (property "Reference" "#PWR0254" (id 0) (at 394.97 96.52 0)
+      (effects (font (size 1.27 1.27)) hide)
+    )
+    (property "Value" "+3V3" (id 1) (at 394.97 87.63 0))
+    (property "Footprint" "" (id 2) (at 394.97 92.71 0)
+      (effects (font (size 1.27 1.27)) hide)
+    )
+    (property "Datasheet" "" (id 3) (at 394.97 92.71 0)
+      (effects (font (size 1.27 1.27)) hide)
+    )
+    (pin "1")
+  )
   (symbol (lib_id "Device:C_Small") (at 57.15 163.83 180) (unit 1)
     (in_bom yes) (on_board yes) (fields_autoplaced)
@@
     (pin "1")
   )
+  (symbol (lib_id "power:PWR_FLAG") (at 408.94 92.71 0) (unit 1)
+    (in_bom yes) (on_board yes) (fields_autoplaced)
+    (property "Reference" "#FLG?" (id 0) (at 408.94 90.805 0)
+      (effects (font (size 1.27 1.27)) hide)
+    )
+    (property "Value" "PWR_FLAG" (id 1) (at 408.94 87.63 0))
+    (property "Footprint" "" (id 2) (at 408.94 92.71 0)
+      (effects (font (size 1.27 1.27)) hide)
+    )
+    (property "Datasheet" "~" (id 3) (at 408.94 92.71 0)
+      (effects (font (size 1.27 1.27)) hide)
+    )
+    (pin "1")
+  )
   (symbol (lib_id "power:+3V3") (at 265.43 96.52 180) (unit 1)
     (in_bom yes) (on_board yes) (fields_autoplaced)
@@
     (pin "1")
   )
+  (symbol (lib_id "power:PWR_FLAG") (at 382.27 95.25 180) (unit 1)
+    (in_bom yes) (on_board yes) (fields_autoplaced)
+    (property "Reference" "#FLG?" (id 0) (at 382.27 97.155 0)
+      (effects (font (size 1.27 1.27)) hide)
+    )
+    (property "Value" "PWR_FLAG" (id 1) (at 382.27 100.33 0))
+    (property "Footprint" "" (id 2) (at 382.27 95.25 0)
+      (effects (font (size 1.27 1.27)) hide)
+    )
+    (property "Datasheet" "~" (id 3) (at 382.27 95.25 0)
+      (effects (font (size 1.27 1.27)) hide)
+    )
+    (pin "1")
+  )
   (symbol (lib_id "marbastlib-mx:MX_SW_HS") (at 463.55 92.71 180) (unit 1)
     (in_bom yes) (on_board yes) (fields_autoplaced)
@@
   )
   (symbol_instances
+    (path "/0bf9f97f-ca31-47aa-9353-faf3444373f3"
+      (reference "#FLG0101") (unit 1) (value "PWR_FLAG") (footprint "")
+    )
+    (path "/0337d994-e584-4621-b400-f84657613a64"
+      (reference "#FLG?") (unit 1) (value "PWR_FLAG") (footprint "")
+    )
+    (path "/abd56bb9-5ea5-4bd5-9568-156170e4da2a"
+      (reference "#FLG?") (unit 1) (value "PWR_FLAG") (footprint "")
+    )
+    (path "/afdaf52e-8fe0-4154-a79b-f79114f8da02"
+      (reference "#FLG?") (unit 1) (value "PWR_FLAG") (footprint "")
+    )
     (path "/aca1f809-f179-492f-82ef-3a9935108ebf"
       (reference "#PWR0101") (unit 1) (value "+3V3") (footprint "")
@@
       (reference "#PWR0253") (unit 1) (value "GND") (footprint "")
     )
+    (path "/55562adf-ef0f-4925-b6a6-26bf7084098f"
+      (reference "#PWR0254") (unit 1) (value "+3V3") (footprint "")
+    )
+    (path "/027f4c19-0a5e-4a64-9c44-0867d88cf5e9"
+      (reference "#PWR?") (unit 1) (value "GND") (footprint "")
+    )
     (path "/6cf076b0-4aa7-48d1-bf18-8a80f7c8ea31"
